Commit message: Reduce to 1 camera and 1 LiDAR in carla_sensor_kit_launch

File: src/carla_sensor_kit_launch/carla_sensor_kit_description/urdf/sensor_kit.xacro (robot description, xacro)
@@ -14,9 +14,11 @@
     - "imu", "inertial" becomes IMU
     - "gnss", "gps" becomes GNSS
-    Sensor List (awsim_labs configuration)
-    - 3 LiDARs (velodyne_top, velodyne_left, velodyne_right)
-    - 8 Cameras (traffic_light_right/left, camera0-5)
+    Sensor List (MINIMAL configuration for performance)
+    - 1 LiDAR (velodyne_top only)
+    - 1 Camera (camera0 front only)
     - 1 GNSS (gnss_link)
     - 1 IMU (tamagawa/imu_link)
+    NOTE - Reduced from full awsim_labs config (3 LiDARs, 8 cameras) to improve
+    CARLA tick rate. See docs/issues-auto-button-disabled.md for details.
     Physical Simulation
     Unlike real sensor kits, these definitions are metadata-only. CARLA handles
@@ -41,4 +43,5 @@
     <!-- LiDAR Sensors -->
     <!-- ========================================================================== -->
+    <!-- MINIMAL CONFIG - Only top LiDAR enabled for performance -->
     <!-- Top LiDAR (VLS-128 equivalent) - Primary 360° coverage -->
     <joint name="velodyne_top_base_link_joint" type="fixed">
@@ -61,83 +64,18 @@
     </joint>
     <link name="velodyne_top"/>
-    <!-- Left LiDAR (VLP-16 equivalent) - Left side coverage -->
+    <!-- DISABLED - Left and Right LiDARs removed for performance
     <joint name="velodyne_left_base_link_joint" type="fixed">
-      <origin
-        xyz="${calibration['sensor_kit_base_link']['velodyne_left_base_link']['x']}
-             ${calibration['sensor_kit_base_link']['velodyne_left_base_link']['y']}
-             ${calibration['sensor_kit_base_link']['velodyne_left_base_link']['z']}"
-        rpy="${calibration['sensor_kit_base_link']['velodyne_left_base_link']['roll']}
-             ${calibration['sensor_kit_base_link']['velodyne_left_base_link']['pitch']}
-             ${calibration['sensor_kit_base_link']['velodyne_left_base_link']['yaw']}"/>
-      <parent link="sensor_kit_base_link"/>
-      <child link="velodyne_left_base_link"/>
+      ...
     </joint>
-    <link name="velodyne_left_base_link"/>
-    <joint name="velodyne_left_joint" type="fixed">
-      <origin xyz="0 0 0" rpy="0 0 0"/>
-      <parent link="velodyne_left_base_link"/>
-      <child link="velodyne_left"/>
+    <joint name="velodyne_right_base_link_joint" type="fixed">
+      ...
     </joint>
-    <link name="velodyne_left"/>
-    <!-- Right LiDAR (VLP-16 equivalent) - Right side coverage -->
-    <joint name="velodyne_right_base_link_joint" type="fixed">
-      <origin
-        xyz="${calibration['sensor_kit_base_link']['velodyne_right_base_link']['x']}
-             ${calibration['sensor_kit_base_link']['velodyne_right_base_link']['y']}
-             ${calibration['sensor_kit_base_link']['velodyne_right_base_link']['z']}"
-        rpy="${calibration['sensor_kit_base_link']['velodyne_right_base_link']['roll']}
-             ${calibration['sensor_kit_base_link']['velodyne_right_base_link']['pitch']}
-             ${calibration['sensor_kit_base_link']['velodyne_right_base_link']['yaw']}"/>
-      <parent link="sensor_kit_base_link"/>
-      <child link="velodyne_right_base_link"/>
-    </joint>
-    <link name="velodyne_right_base_link"/>
-    <joint name="velodyne_right_joint" type="fixed">
-      <origin xyz="0 0 0" rpy="0 0 0"/>
-      <parent link="velodyne_right_base_link"/>
-      <child link="velodyne_right"/>
-    </joint>
-    <link name="velodyne_right"/>
+    -->
     <!-- ========================================================================== -->
     <!-- Camera Sensors -->
     <!-- ========================================================================== -->
-    <!-- Traffic Light Recognition Cameras -->
-    <joint name="traffic_light_right_camera_link_joint" type="fixed">
-      <origin
-        xyz="${calibration['sensor_kit_base_link']['traffic_light_right_camera/camera_link']['x']}
-             ${calibration['sensor_kit_base_link']['traffic_light_right_camera/camera_link']['y']}
-             ${calibration['sensor_kit_base_link']['traffic_light_right_camera/camera_link']['z']}"
-        rpy="${calibration['sensor_kit_base_link']['traffic_light_right_camera/camera_link']['roll']}
-             ${calibration['sensor_kit_base_link']['traffic_light_right_camera/camera_link']['pitch']}
-             ${calibration['sensor_kit_base_link']['traffic_light_right_camera/camera_link']['yaw']}"/>
-      <parent link="sensor_kit_base_link"/>
-      <child link="traffic_light_right_camera/camera_link"/>
-    </joint>
-    <link name="traffic_light_right_camera/camera_link"/>
-    <joint name="traffic_light_right_camera_optical_link_joint" type="fixed">
-      <origin xyz="0 0 0" rpy="-1.5707963267948966 0 -1.5707963267948966"/>
-      <parent link="traffic_light_right_camera/camera_link"/>
-      <child link="traffic_light_right_camera/camera_optical_link"/>
-    </joint>
-    <link name="traffic_light_right_camera/camera_optical_link"/>
-    <joint name="traffic_light_left_camera_link_joint" type="fixed">
-      <origin
-        xyz="${calibration['sensor_kit_base_link']['traffic_light_left_camera/camera_link']['x']}
-             ${calibration['sensor_kit_base_link']['traffic_light_left_camera/camera_link']['y']}
-             ${calibration['sensor_kit_base_link']['traffic_light_left_camera/camera_link']['z']}"
-        rpy="${calibration['sensor_kit_base_link']['traffic_light_left_camera/camera_link']['roll']}
-             ${calibration['sensor_kit_base_link']['traffic_light_left_camera/camera_link']['pitch']}
-             ${calibration['sensor_kit_base_link']['traffic_light_left_camera/camera_link']['yaw']}"/>
-      <parent link="sensor_kit_base_link"/>
-      <child link="traffic_light_left_camera/camera_link"/>
-    </joint>
-    <link name="traffic_light_left_camera/camera_link"/>
-    <joint name="traffic_light_left_camera_optical_link_joint" type="fixed">
-      <origin xyz="0 0 0" rpy="-1.5707963267948966 0 -1.5707963267948966"/>
-      <parent link="traffic_light_left_camera/camera_link"/>
-      <child link="traffic_light_left_camera/camera_optical_link"/>
-    </joint>
-    <link name="traffic_light_left_camera/camera_optical_link"/>
-    <!-- Surround View Cameras (camera0-5) -->
+    <!-- MINIMAL CONFIG - Only camera0 (front) enabled for performance -->
+    <!-- DISABLED - Traffic Light Recognition Cameras removed for performance -->
+    <!-- Surround View Cameras - Only camera0 enabled -->
     <xacro:macro name="surround_camera" params="name">
       <!-- Build the calibration key name -->
@@ -163,5 +101,7 @@
       <link name="${name}/camera_optical_link"/>
     </xacro:macro>
+    <!-- Only front camera enabled -->
     <xacro:surround_camera name="camera0"/>
+    <!-- DISABLED - camera1-5 removed for performance
     <xacro:surround_camera name="camera1"/>
     <xacro:surround_camera name="camera2"/>
@@ -169,4 +109,5 @@
     <xacro:surround_camera name="camera4"/>
     <xacro:surround_camera name="camera5"/>
+    -->
     <!-- ========================================================================== -->
     <!-- GNSS Sensor -->

Commit message: [carla_sensor_kit_launch] Fix frame names and topic names

File: src/carla_sensor_kit_launch/carla_sensor_kit_description/urdf/sensor_kit.xacro (robot description, xacro)
@@ -45,5 +45,6 @@
     <!-- MINIMAL CONFIG - Only top LiDAR enabled for performance -->
     <!-- Top LiDAR (VLS-128 equivalent) - Primary 360° coverage -->
-    <joint name="velodyne_top_base_link_joint" type="fixed">
+    <!-- Named "top" to match Autoware's expected topic namespace /sensing/lidar/top/... -->
+    <joint name="top_base_link_joint" type="fixed">
       <origin
         xyz="${calibration['sensor_kit_base_link']['velodyne_top_base_link']['x']}
@@ -54,14 +55,14 @@
              ${calibration['sensor_kit_base_link']['velodyne_top_base_link']['yaw']}"/>
       <parent link="sensor_kit_base_link"/>
-      <child link="velodyne_top_base_link"/>
+      <child link="top_base_link"/>
     </joint>
-    <link name="velodyne_top_base_link"/>
+    <link name="top_base_link"/>
     <!-- Actual sensor frame (optical frame) -->
-    <joint name="velodyne_top_joint" type="fixed">
+    <joint name="top_joint" type="fixed">
       <origin xyz="0 0 0" rpy="0 0 0"/>
-      <parent link="velodyne_top_base_link"/>
-      <child link="velodyne_top"/>
+      <parent link="top_base_link"/>
+      <child link="top"/>
     </joint>
-    <link name="velodyne_top"/>
+    <link name="top"/>
     <!-- DISABLED - Left and Right LiDARs removed for performance
     <joint name="velodyne_left_base_link_joint" type="fixed">
@@ -113,31 +114,31 @@
     <!-- GNSS Sensor -->
     <!-- ========================================================================== -->
-    <joint name="gnss_link_joint" type="fixed">
+    <joint name="carla_gnss_link_joint" type="fixed">
       <origin
-        xyz="${calibration['sensor_kit_base_link']['gnss_link']['x']}
-             ${calibration['sensor_kit_base_link']['gnss_link']['y']}
-             ${calibration['sensor_kit_base_link']['gnss_link']['z']}"
-        rpy="${calibration['sensor_kit_base_link']['gnss_link']['roll']}
-             ${calibration['sensor_kit_base_link']['gnss_link']['pitch']}
-             ${calibration['sensor_kit_base_link']['gnss_link']['yaw']}"/>
+        xyz="${calibration['sensor_kit_base_link']['carla/gnss_link']['x']}
+             ${calibration['sensor_kit_base_link']['carla/gnss_link']['y']}
+             ${calibration['sensor_kit_base_link']['carla/gnss_link']['z']}"
+        rpy="${calibration['sensor_kit_base_link']['carla/gnss_link']['roll']}
+             ${calibration['sensor_kit_base_link']['carla/gnss_link']['pitch']}
+             ${calibration['sensor_kit_base_link']['carla/gnss_link']['yaw']}"/>
       <parent link="sensor_kit_base_link"/>
-      <child link="gnss_link"/>
+      <child link="carla/gnss_link"/>
     </joint>
-    <link name="gnss_link"/>
+    <link name="carla/gnss_link"/>
     <!-- ========================================================================== -->
     <!-- IMU Sensor -->
     <!-- ========================================================================== -->
-    <joint name="tamagawa_imu_link_joint" type="fixed">
+    <joint name="carla_imu_link_joint" type="fixed">
       <origin
-        xyz="${calibration['sensor_kit_base_link']['tamagawa/imu_link']['x']}
-             ${calibration['sensor_kit_base_link']['tamagawa/imu_link']['y']}
-             ${calibration['sensor_kit_base_link']['tamagawa/imu_link']['z']}"
-        rpy="${calibration['sensor_kit_base_link']['tamagawa/imu_link']['roll']}
-             ${calibration['sensor_kit_base_link']['tamagawa/imu_link']['pitch']}
-             ${calibration['sensor_kit_base_link']['tamagawa/imu_link']['yaw']}"/>
+        xyz="${calibration['sensor_kit_base_link']['carla/imu_link']['x']}
+             ${calibration['sensor_kit_base_link']['carla/imu_link']['y']}
+             ${calibration['sensor_kit_base_link']['carla/imu_link']['z']}"
+        rpy="${calibration['sensor_kit_base_link']['carla/imu_link']['roll']}
+             ${calibration['sensor_kit_base_link']['carla/imu_link']['pitch']}
+             ${calibration['sensor_kit_base_link']['carla/imu_link']['yaw']}"/>
       <parent link="sensor_kit_base_link"/>
-      <child link="tamagawa/imu_link"/>
+      <child link="carla/imu_link"/>
     </joint>
-    <link name="tamagawa/imu_link"/>
+    <link name="carla/imu_link"/>
   </xacro:macro>
 </robot>

File: src/carla_sensor_kit_launch/carla_sensor_kit_description/urdf/sensors.xacro (robot description, xacro)
@@ -14,15 +14,8 @@
     yaw="${calibration['base_link']['sensor_kit_base_link']['yaw']}"
   />
-  <!-- embedded sensors -->
-  <xacro:include filename="$(find velodyne_description)/urdf/VLP-16.urdf.xacro"/>
-  <xacro:VLP-16 parent="base_link" name="velodyne_rear" topic="velodyne_rear/velodyne_points" hz="10" samples="220" gpu="false">
-    <origin
-      xyz="${calibration['base_link']['velodyne_rear_base_link']['x']}
-           ${calibration['base_link']['velodyne_rear_base_link']['y']}
-           ${calibration['base_link']['velodyne_rear_base_link']['z']}"
-      rpy="${calibration['base_link']['velodyne_rear_base_link']['roll']}
-           ${calibration['base_link']['velodyne_rear_base_link']['pitch']}
-           ${calibration['base_link']['velodyne_rear_base_link']['yaw']}"
-    />
-  </xacro:VLP-16>
+  <!--
+    NOTE - embedded sensors (velodyne_rear) removed for CARLA simulation
+    CARLA uses the 'top' LiDAR defined in sensor_kit.xacro with matching topic names
+    for Autoware's pointcloud_preprocessor pipeline.
+  -->
 </robot>
