Commit message: feat(sensors): IMU and GNSS frames are imu_link and gnss_link
The CARLA sensor kit's IMU and GNSS frames were carla/imu_link and
carla/gnss_link, names aib (the Isaac bridge) inherited by reusing this sensing
layout. They are now simulator-neutral: frames imu_link and gnss_link, and so
(the bridge derives the topic from the sensor name) topics
/sensing/imu/imu_link/imu_raw and /sensing/gnss/gnss_link/nav_sat_fix. aib
renames its spec in step.

Changed together: vehicle_config.yaml's sensor keys (the frame_id and topic
acb_bridge publishes), the sensor kit's calibration (both copies) and xacro
links and joints, and the sensing launch. imu.launch.xml and gnss.launch.xml
take the topic as an argument (imu_raw_name, gnss_fix_name, as Autoware's
sample kit does) instead of naming it twice.

Nothing in Autoware 1.5.0 assumes a vendor/imu_link frame: imu_corrector and
gyro_odometer go through TF from the message's frame_id.

Co-Authored-By: Claude Opus 5.5 <noreply@anthropic.com>
Claude-Session: https://claude.ai/code/session_01XsykZth51hsT5oMxxVHcNK

File: src/acb_sensor_kit_launch/acb_sensor_kit_description/urdf/sensor_kit.xacro (robot description, xacro)
@@ -18,5 +18,5 @@
     - 1 Camera (camera0 front only)
     - 1 GNSS (gnss_link)
-    - 1 IMU (tamagawa/imu_link)
+    - 1 IMU (imu_link)
     NOTE - Reduced from full awsim_labs config (3 LiDARs, 8 cameras) to improve
     CARLA tick rate. See docs/issues-auto-button-disabled.md for details.
@@ -118,31 +118,31 @@
     <!-- GNSS Sensor -->
     <!-- ========================================================================== -->
-    <joint name="carla_gnss_link_joint" type="fixed">
+    <joint name="gnss_link_joint" type="fixed">
       <origin
-        xyz="${calibration['sensor_kit_base_link']['carla/gnss_link']['x']}
-             ${calibration['sensor_kit_base_link']['carla/gnss_link']['y']}
-             ${calibration['sensor_kit_base_link']['carla/gnss_link']['z']}"
-        rpy="${calibration['sensor_kit_base_link']['carla/gnss_link']['roll']}
-             ${calibration['sensor_kit_base_link']['carla/gnss_link']['pitch']}
-             ${calibration['sensor_kit_base_link']['carla/gnss_link']['yaw']}"/>
+        xyz="${calibration['sensor_kit_base_link']['gnss_link']['x']}
+             ${calibration['sensor_kit_base_link']['gnss_link']['y']}
+             ${calibration['sensor_kit_base_link']['gnss_link']['z']}"
+        rpy="${calibration['sensor_kit_base_link']['gnss_link']['roll']}
+             ${calibration['sensor_kit_base_link']['gnss_link']['pitch']}
+             ${calibration['sensor_kit_base_link']['gnss_link']['yaw']}"/>
       <parent link="sensor_kit_base_link"/>
-      <child link="carla/gnss_link"/>
+      <child link="gnss_link"/>
     </joint>
-    <link name="carla/gnss_link"/>
+    <link name="gnss_link"/>
     <!-- ========================================================================== -->
     <!-- IMU Sensor -->
     <!-- ========================================================================== -->
-    <joint name="carla_imu_link_joint" type="fixed">
+    <joint name="imu_link_joint" type="fixed">
       <origin
-        xyz="${calibration['sensor_kit_base_link']['carla/imu_link']['x']}
-             ${calibration['sensor_kit_base_link']['carla/imu_link']['y']}
-             ${calibration['sensor_kit_base_link']['carla/imu_link']['z']}"
-        rpy="${calibration['sensor_kit_base_link']['carla/imu_link']['roll']}
-             ${calibration['sensor_kit_base_link']['carla/imu_link']['pitch']}
-             ${calibration['sensor_kit_base_link']['carla/imu_link']['yaw']}"/>
+        xyz="${calibration['sensor_kit_base_link']['imu_link']['x']}
+             ${calibration['sensor_kit_base_link']['imu_link']['y']}
+             ${calibration['sensor_kit_base_link']['imu_link']['z']}"
+        rpy="${calibration['sensor_kit_base_link']['imu_link']['roll']}
+             ${calibration['sensor_kit_base_link']['imu_link']['pitch']}
+             ${calibration['sensor_kit_base_link']['imu_link']['yaw']}"/>
       <parent link="sensor_kit_base_link"/>
-      <child link="carla/imu_link"/>
+      <child link="imu_link"/>
     </joint>
-    <link name="carla/imu_link"/>
+    <link name="imu_link"/>
   </xacro:macro>
 </robot>
